File: R_OlivaTPFinal/WEMB02_j/WEMB02_j/WEMB02_j.sch (KiCad schematic (older format))
At the start: 7 parts

Commit message: WEMB02-J Sch + PCB completos, faltan algunos mod.3D
Other:
- note added: "PLACA MADRE - WIND EMPOWERMENT WEMB02\nCONTROL Y ALIMENTACION MÓDULOS DE POTENCIA\nPARA SOLAR / EOLICA\nREV. WEMB02J - R.OLIVA 8.12.2018\n"
Changed lines of the file:
@@
 L Mechanical:MountingHole MH101
 U 1 1 5BE412CE
-P 2350 5750
-F 0 "MH101" H 2450 5796 50  0000 L CNN
-F 1 "MH4mm" H 2450 5705 50  0000 L CNN
-F 2 "MountingHole:MountingHole_4mm" H 2350 5750 50  0001 C CNN
-F 3 "~" H 2350 5750 50  0001 C CNN
-	1    2350 5750
+P 2350 5800
+F 0 "MH101" H 2450 5846 50  0000 L CNN
+F 1 "MH4mm" H 2450 5755 50  0000 L CNN
+F 2 "MountingHole:MountingHole_4mm" H 2350 5800 50  0001 C CNN
+F 3 "~" H 2350 5800 50  0001 C CNN
+	1    2350 5800
 	1    0    0    -1
 $EndComp
@@
 L Mechanical:MountingHole MH102
 U 1 1 5BE4135A
-P 2900 5750
-F 0 "MH102" H 3000 5796 50  0000 L CNN
-F 1 "MH4mm" H 3000 5705 50  0000 L CNN
-F 2 "MountingHole:MountingHole_4mm" H 2900 5750 50  0001 C CNN
-F 3 "~" H 2900 5750 50  0001 C CNN
-	1    2900 5750
+P 2900 5800
+F 0 "MH102" H 3000 5846 50  0000 L CNN
+F 1 "MH4mm" H 3000 5755 50  0000 L CNN
+F 2 "MountingHole:MountingHole_4mm" H 2900 5800 50  0001 C CNN
+F 3 "~" H 2900 5800 50  0001 C CNN
+	1    2900 5800
 	1    0    0    -1
 $EndComp
@@
 L Mechanical:MountingHole MH103
 U 1 1 5BE41388
-P 3450 5750
-F 0 "MH103" H 3550 5796 50  0000 L CNN
-F 1 "MH4mm" H 3550 5705 50  0000 L CNN
-F 2 "MountingHole:MountingHole_4mm" H 3450 5750 50  0001 C CNN
-F 3 "~" H 3450 5750 50  0001 C CNN
-	1    3450 5750
+P 3450 5800
+F 0 "MH103" H 3550 5846 50  0000 L CNN
+F 1 "MH4mm" H 3550 5755 50  0000 L CNN
+F 2 "MountingHole:MountingHole_4mm" H 3450 5800 50  0001 C CNN
+F 3 "~" H 3450 5800 50  0001 C CNN
+	1    3450 5800
 	1    0    0    -1
 $EndComp
@@
 L Mechanical:MountingHole MH104
 U 1 1 5BE413B0
-P 4000 5750
-F 0 "MH104" H 4100 5796 50  0000 L CNN
-F 1 "MH4mm" H 4100 5700 50  0000 L CNN
-F 2 "MountingHole:MountingHole_4mm" H 4000 5750 50  0001 C CNN
-F 3 "~" H 4000 5750 50  0001 C CNN
-	1    4000 5750
+P 4000 5800
+F 0 "MH104" H 4100 5846 50  0000 L CNN
+F 1 "MH4mm" H 4100 5750 50  0000 L CNN
+F 2 "MountingHole:MountingHole_4mm" H 4000 5800 50  0001 C CNN
+F 3 "~" H 4000 5800 50  0001 C CNN
+	1    4000 5800
 	1    0    0    -1
 $EndComp
@@
 L Mechanical:MountingHole F101
 U 1 1 5BE442B8
-P 2350 6250
-F 0 "F101" H 2450 6296 50  0000 L CNN
-F 1 "Fiducial" H 2450 6205 50  0000 L CNN
-F 2 "Fiducial:Fiducial_1mm_Dia_2mm_Outer" H 2350 6250 50  0001 C CNN
-F 3 "~" H 2350 6250 50  0001 C CNN
-	1    2350 6250
+P 2350 6300
+F 0 "F101" H 2450 6346 50  0000 L CNN
+F 1 "Fiducial" H 2450 6255 50  0000 L CNN
+F 2 "Fiducial:Fiducial_1mm_Dia_2mm_Outer" H 2350 6300 50  0001 C CNN
+F 3 "~" H 2350 6300 50  0001 C CNN
+	1    2350 6300
 	1    0    0    -1
 $EndComp
@@
 L Mechanical:MountingHole F102
 U 1 1 5BE44331
-P 2900 6250
-F 0 "F102" H 3000 6296 50  0000 L CNN
-F 1 "Fiducial" H 3000 6205 50  0000 L CNN
-F 2 "Fiducial:Fiducial_1mm_Dia_2mm_Outer" H 2900 6250 50  0001 C CNN
-F 3 "~" H 2900 6250 50  0001 C CNN
-	1    2900 6250
+P 2900 6300
+F 0 "F102" H 3000 6346 50  0000 L CNN
+F 1 "Fiducial" H 3000 6255 50  0000 L CNN
+F 2 "Fiducial:Fiducial_1mm_Dia_2mm_Outer" H 2900 6300 50  0001 C CNN
+F 3 "~" H 2900 6300 50  0001 C CNN
+	1    2900 6300
 	1    0    0    -1
 $EndComp
@@
 L Mechanical:MountingHole F103
 U 1 1 5BE6EFCC
-P 3450 6250
-F 0 "F103" H 3550 6296 50  0000 L CNN
-F 1 "Fiducial" H 3550 6205 50  0000 L CNN
-F 2 "Fiducial:Fiducial_1mm_Dia_2mm_Outer" H 3450 6250 50  0001 C CNN
-F 3 "~" H 3450 6250 50  0001 C CNN
-	1    3450 6250
+P 3450 6300
+F 0 "F103" H 3550 6346 50  0000 L CNN
+F 1 "Fiducial" H 3550 6255 50  0000 L CNN
+F 2 "Fiducial:Fiducial_1mm_Dia_2mm_Outer" H 3450 6300 50  0001 C CNN
+F 3 "~" H 3450 6300 50  0001 C CNN
+	1    3450 6300
 	1    0    0    -1
 $EndComp
@@
 Wire Wire Line
 	3350 4000 4350 4000
+Text Notes 4100 1500 0    79   ~ 16
+PLACA MADRE - WIND EMPOWERMENT WEMB02\nCONTROL Y ALIMENTACION MÓDULOS DE POTENCIA\nPARA SOLAR / EOLICA\nREV. WEMB02J - R.OLIVA 8.12.2018\n
+Wire Notes Line
+	4050 900  7150 900
+Wire Notes Line
+	7150 900  7150 1600
+Wire Notes Line
+	7150 1600 4050 1600
+Wire Notes Line
+	4050 1600 4050 900
 $EndSCHEMATC
