File: R_OlivaTPFinal/WEMB02_j/WEMB02_j/power.sch (KiCad schematic (older format))
At the start: 39 parts, among them J301 EXP_PWR, Q301 BC817-40_215, Q302 BC817-40_215, U301 SDM30-125S, U302 FEEDER_BRD, U303 R-78E3.3-0.5, U304 R-78E5.0-1.0

Commit message: WEMB02-J Sch + PCB completos, faltan algunos mod.3D
Changed lines of the file:
@@
 Wire Notes Line
 	6850 3200 6850 7500
-Text Notes 5200 2850 0    79   ~ 16
+Text Notes 5200 2800 0    79   ~ 16
 MODULO FEEDER\nPRINCIPAL  +15V\n
 Text Notes 8350 2850 0    79   ~ 16
